File: KiCAD_DRONE/Drone_rev0/ESC_rev1/ESC_rev1/ESC_rev1.sch (KiCad schematic (older format))
At the start: 34 parts, among them J1 Conn_01x02, J2 Conn_01x06, J3 Conn_01x05, Q1 IRF3205, Q2 IRF3205, Q3 IRF3205, Q4 IRF3205, Q5 IRF3205, Q6 IRF3205, U1 LM27222, U2 LM27222, U3 LM27222

Commit message: finished ESC rev1 layout!
Parts:
- removed J3: Conn_01x05, Connector_PinHeader_2.54mm:PinHeader_1x05_P2.54mm_Vertical, symbol Connector_Generic:Conn_01x05
- added C14, C15, C16: C, Capacitor_SMD:C_0805_2012Metric, symbol Device:C
- added J3: Conn_01x07, Connector_PinHeader_2.54mm:PinHeader_1x07_P2.54mm_Vertical, symbol Connector_Generic:Conn_01x07
- added J4, J5, J6: Conn_01x02, Connector_JST:JST_EH_B02B-EH-A_1x02_P2.50mm_Vertical, symbol Connector_Generic:Conn_01x02
- added R10, R11, R12, R13, R14, R15, R7, R8, R9: R, Resistor_SMD:R_0805_2012Metric, symbol Device:R
Connections:
- net GND: now also C1.2; no longer C1.1, U1.8 (GND), U2.8 (GND), U3.8 (GND)
- net Vcc: now also C1.1; no longer C1.2, D1.2 (A), D2.2 (A), D3.2 (A), U1.6 (Vcc), U2.6 (Vcc), U3.6 (Vcc)
- net at C2.1, U1.1 (SW): now also C5.2, Q1.3 (S), Q2.2 (D), R1.2, J3.1 (Pin_1)
- net at U1.2 (HG): now also R8.2; no longer Q1.1 (G)
- net at U1.7 (LG): now also R9.2; no longer Q2.1 (G)
- net at Q3.1 (G): now also R11.1; no longer U2.2 (HG)
- net at C6.1, C9.2, Q3.3 (S)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: now also J3.3 (Pin_3)
- net at Q4.1 (G): now also R12.1; no longer U2.7 (LG)
- net at Q5.1 (G): now also R14.1; no longer U3.2 (HG)
- net at C10.1, C12.2, Q5.3 (S)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: now also J3.5 (Pin_5)
- net at Q6.1 (G): now also R15.1; no longer U3.7 (LG)
- new net: D1.2 (A), R7.1, U1.6 (Vcc)
- new net: Q1.1 (G), R8.1
- new net: Q2.1 (G), R9.1
- new net: R11.2, U2.2 (HG)
- new net: D2.2 (A), R10.1, U2.6 (Vcc)
- new net: R12.2, U2.7 (LG)
- new net: R14.2, U3.2 (HG)
- new net: D3.2 (A), R13.1, U3.6 (Vcc)
- new net: R15.2, U3.7 (LG)
- new net VDD1: C14.1, J4.2 (Pin_2), R7.2
- new net VDD2: C15.1, J5.2 (Pin_2), R10.2
- new net VDD3: C16.1, J6.2 (Pin_2), R13.2
- new net VSS1: C14.2, J4.1 (Pin_1), U1.8 (GND)
- new net VSS2: C15.2, J5.1 (Pin_1), U2.8 (GND)
- new net VSS3: C16.2, J6.1 (Pin_1), U3.8 (GND)
- no-connect marks 2 -> 4
Other:
- moved on the sheet: C1, J1, J2
