File: KiCAD_DRONE/Drone_rev0/ESC_rev1/ESC_rev1/ESC_rev1.sch (KiCad schematic (older format))
At the start: 49 parts, among them J1 Conn_01x02, J2 Conn_01x06, J3 Conn_01x07, J4 Conn_01x02, J5 Conn_01x02, J6 Conn_01x02, Q1 IRF3205, Q2 IRF3205, Q3 IRF3205, Q4 IRF3205, Q5 IRF3205, Q6 IRF3205, U1 LM27222, U2 LM27222, U3 LM27222

Commit message: added text and final layout changes. added m60 files.
Parts:
- removed J2: Conn_01x06, Connector_PinHeader_2.54mm:PinHeader_1x06_P2.54mm_Vertical, symbol Connector_Generic:Conn_01x06
- added J2: Conn_01x07, Connector_JST:JST_EH_B07B-EH-A_1x07_P2.50mm_Vertical, symbol Connector_Generic:Conn_01x07
Connections:
- net VSS2 is gone; now on net VSS1: C15.2, J5.1 (Pin_1), U2.8 (GND)
- net VSS3 is gone; now on net VSS1: C16.2, J6.1 (Pin_1), U3.8 (GND)
- net AH: now also J2.4 (Pin_4)
- net AL: now also J2.7 (Pin_7)
- net BH: now also J2.3 (Pin_3)
- net BL: now also J2.6 (Pin_6)
- net CH: now also J2.2 (Pin_2)
- net CL: now also J2.5 (Pin_5)
- net VSS1: now also J2.1 (Pin_1)
Changed lines of the file:
@@
 	6700 5800 6700 6000
 Connection ~ 6700 5800
-Text GLabel 4100 4100 2    50   Output ~ 0
+Text GLabel 4100 3950 2    50   Output ~ 0
 AL
-Text GLabel 4100 4200 2    50   Output ~ 0
+Text GLabel 4100 4050 2    50   Output ~ 0
 BL
 Wire Wire Line
-	3850 4100 4100 4100
-Wire Wire Line
-	3850 4200 4100 4200
+	3850 3950 4100 3950
+Wire Wire Line
+	3850 4050 4100 4050
 $Comp
 L My_Schematics:LM27222 U2
@@
 Text GLabel 7650 5650 0    50   Input ~ 0
 BL
-Text GLabel 4100 4400 2    50   Output ~ 0
+Text GLabel 4100 4250 2    50   Output ~ 0
 AH
 Wire Wire Line
-	3850 4400 4100 4400
+	3850 4250 4100 4250
 Wire Wire Line
 	4900 4650 5150 4650
@@
 Wire Wire Line
 	7650 5650 7850 5650
-Text GLabel 4100 4500 2    50   Output ~ 0
+Text GLabel 4100 4350 2    50   Output ~ 0
 BH
 Wire Wire Line
-	3850 4500 4100 4500
+	3850 4350 4100 4350
 Text GLabel 7650 5750 0    50   Input ~ 0
 BH
@@
 Wire Wire Line
 	6700 4600 6700 4750
-Text GLabel 4100 4600 2    50   Output ~ 0
+Text GLabel 4100 4450 2    50   Output ~ 0
 CH
-Text GLabel 4100 4300 2    50   Output ~ 0
+Text GLabel 4100 4150 2    50   Output ~ 0
 CL
 Wire Wire Line
-	3850 4300 4100 4300
-Wire Wire Line
-	3850 4600 4100 4600
-$Comp
-L Connector_Generic:Conn_01x06 J2
-U 1 1 5CEE7D4C
-P 3650 4400
-F 0 "J2" H 3570 3875 50  0000 C CNN
-F 1 "Conn_01x06" H 3570 3966 50  0000 C CNN
-F 2 "Connector_PinHeader_2.54mm:PinHeader_1x06_P2.54mm_Vertical" H 3650 4400 50  0001 C CNN
-F 3 "~" H 3650 4400 50  0001 C CNN
-	1    3650 4400
-	-1   0    0    1
-$EndComp
+	3850 4150 4100 4150
+Wire Wire Line
+	3850 4450 4100 4450
 NoConn ~ 13350 4650
 NoConn ~ 13350 4850
@@
 Text GLabel 4050 6000 2    50   Output ~ 0
 VDD3
-Text GLabel 4050 5700 2    50   Output ~ 0
-VSS2
-Text GLabel 4050 6300 2    50   Output ~ 0
-VSS3
 Wire Wire Line
 	3850 3200 3850 3500
@@
 Text GLabel 7550 5150 0    50   Input ~ 0
 VDD2
-Text GLabel 7850 5850 0    50   Input ~ 0
-VSS2
 Text GLabel 10050 5150 0    50   Input ~ 0
 VDD3
-Text GLabel 10350 5850 0    50   Input ~ 0
-VSS3
 $Comp
 L Device:R R8
@@
 NoConn ~ 13350 5050
 NoConn ~ 13350 5150
+$Comp
+L Connector_Generic:Conn_01x07 J2
+U 1 1 5D02E0AC
+P 3650 4250
+F 0 "J2" H 3570 3725 50  0000 C CNN
+F 1 "Conn_01x07" H 3570 3816 50  0000 C CNN
+F 2 "Connector_JST:JST_EH_B07B-EH-A_1x07_P2.50mm_Vertical" H 3650 4250 50  0001 C CNN
+F 3 "~" H 3650 4250 50  0001 C CNN
+	1    3650 4250
+	-1   0    0    1
+$EndComp
+Text GLabel 3850 4550 2    50   Output ~ 0
+VSS1
+Text GLabel 4050 5700 2    50   Output ~ 0
+VSS1
+Text GLabel 4050 6300 2    50   Output ~ 0
+VSS1
+Text GLabel 7850 5850 0    50   Input ~ 0
+VSS1
+Text GLabel 10350 5850 0    50   Input ~ 0
+VSS1
 $EndSCHEMATC

Commit message: added documents
Parts:
- C1, C13, C14, C15, C16, C3, C7: value C -> 100n
- C10, C2, C6: value C -> .22u
- C11, C12, C4, C5, C8, C9: value C -> 390p
- R1, R2, R3, R4, R5, R6: value R -> 5.1
- R10, R13, R7: value R -> 10
- R11, R12, R14, R15, R8, R9: value R -> 12
Changed lines of the file:
@@
 P 5950 4400
 F 0 "C2" V 5698 4400 50  0000 C CNN
-F 1 "C" V 5789 4400 50  0000 C CNN
+F 1 ".22u" V 5789 4400 50  0000 C CNN
 F 2 "Capacitor_SMD:C_0805_2012Metric" H 5988 4250 50  0001 C CNN
 F 3 "~" H 5950 4400 50  0001 C CNN
@@
 P 4000 3200
 F 0 "C1" H 3885 3154 50  0000 R CNN
-F 1 "C" H 3885 3245 50  0000 R CNN
+F 1 "100n" H 3885 3245 50  0000 R CNN
 F 2 "Capacitor_SMD:C_0805_2012Metric" H 4038 3050 50  0001 C CNN
 F 3 "~" H 4000 3200 50  0001 C CNN
@@
 P 7000 3550
 F 0 "C3" H 6885 3504 50  0000 R CNN
-F 1 "C" H 6885 3595 50  0000 R CNN
+F 1 "100n" H 6885 3595 50  0000 R CNN
 F 2 "Capacitor_SMD:C_0805_2012Metric" H 7038 3400 50  0001 C CNN
 F 3 "~" H 7000 3550 50  0001 C CNN
@@
 P 9700 3500
 F 0 "C7" H 9585 3454 50  0000 R CNN
-F 1 "C" H 9585 3545 50  0000 R CNN
+F 1 "100n" H 9585 3545 50  0000 R CNN
 F 2 "Capacitor_SMD:C_0805_2012Metric" H 9738 3350 50  0001 C CNN
 F 3 "~" H 9700 3500 50  0001 C CNN
@@
 P 12250 3500
 F 0 "C13" H 12135 3454 50  0000 R CNN
-F 1 "C" H 12135 3545 50  0000 R CNN
+F 1 "100n" H 12135 3545 50  0000 R CNN
 F 2 "Capacitor_SMD:C_0805_2012Metric" H 12288 3350 50  0001 C CNN
 F 3 "~" H 12250 3500 50  0001 C CNN
@@
 P 7050 4150
 F 0 "C4" H 6935 4104 50  0000 R CNN
-F 1 "C" H 6935 4195 50  0000 R CNN
+F 1 "390p" H 6935 4195 50  0000 R CNN
 F 2 "Capacitor_SMD:C_0805_2012Metric" H 7088 4000 50  0001 C CNN
 F 3 "~" H 7050 4150 50  0001 C CNN
@@
 P 7050 4450
 F 0 "R1" H 7120 4496 50  0000 L CNN
-F 1 "R" H 7120 4405 50  0000 L CNN
+F 1 "5.1" H 7120 4405 50  0000 L CNN
 F 2 "Resistor_SMD:R_0805_2012Metric" V 6980 4450 50  0001 C CNN
 F 3 "~" H 7050 4450 50  0001 C CNN
@@
 P 7050 5350
 F 0 "C5" H 6935 5304 50  0000 R CNN
-F 1 "C" H 6935 5395 50  0000 R CNN
+F 1 "390p" H 6935 5395 50  0000 R CNN
 F 2 "Capacitor_SMD:C_0805_2012Metric" H 7088 5200 50  0001 C CNN
 F 3 "~" H 7050 5350 50  0001 C CNN
@@
 P 7050 5650
 F 0 "R2" H 7120 5696 50  0000 L CNN
-F 1 "R" H 7120 5605 50  0000 L CNN
+F 1 "5.1" H 7120 5605 50  0000 L CNN
 F 2 "Resistor_SMD:R_0805_2012Metric" V 6980 5650 50  0001 C CNN
 F 3 "~" H 7050 5650 50  0001 C CNN
@@
 P 9700 4100
 F 0 "C8" H 9585 4054 50  0000 R CNN
-F 1 "C" H 9585 4145 50  0000 R CNN
+F 1 "390p" H 9585 4145 50  0000 R CNN
 F 2 "Capacitor_SMD:C_0805_2012Metric" H 9738 3950 50  0001 C CNN
 F 3 "~" H 9700 4100 50  0001 C CNN
@@
 P 9700 4400
 F 0 "R3" H 9770 4446 50  0000 L CNN
-F 1 "R" H 9770 4355 50  0000 L CNN
+F 1 "5.1" H 9770 4355 50  0000 L CNN
 F 2 "Resistor_SMD:R_0805_2012Metric" V 9630 4400 50  0001 C CNN
 F 3 "~" H 9700 4400 50  0001 C CNN
@@
 P 12200 4100
 F 0 "C11" H 12085 4054 50  0000 R CNN
-F 1 "C" H 12085 4145 50  0000 R CNN
+F 1 "390p" H 12085 4145 50  0000 R CNN
 F 2 "Capacitor_SMD:C_0805_2012Metric" H 12238 3950 50  0001 C CNN
 F 3 "~" H 12200 4100 50  0001 C CNN
@@
 P 12200 4400
 F 0 "R5" H 12270 4446 50  0000 L CNN
-F 1 "R" H 12270 4355 50  0000 L CNN
+F 1 "5.1" H 12270 4355 50  0000 L CNN
 F 2 "Resistor_SMD:R_0805_2012Metric" V 12130 4400 50  0001 C CNN
 F 3 "~" H 12200 4400 50  0001 C CNN
@@
 P 9700 5300
 F 0 "C9" H 9585 5254 50  0000 R CNN
-F 1 "C" H 9585 5345 50  0000 R CNN
+F 1 "390p" H 9585 5345 50  0000 R CNN
 F 2 "Capacitor_SMD:C_0805_2012Metric" H 9738 5150 50  0001 C CNN
 F 3 "~" H 9700 5300 50  0001 C CNN
@@
 P 9700 5600
 F 0 "R4" H 9770 5646 50  0000 L CNN
-F 1 "R" H 9770 5555 50  0000 L CNN
+F 1 "5.1" H 9770 5555 50  0000 L CNN
 F 2 "Resistor_SMD:R_0805_2012Metric" V 9630 5600 50  0001 C CNN
 F 3 "~" H 9700 5600 50  0001 C CNN
@@
 P 12200 5300
 F 0 "C12" H 12085 5254 50  0000 R CNN
-F 1 "C" H 12085 5345 50  0000 R CNN
+F 1 "390p" H 12085 5345 50  0000 R CNN
 F 2 "Capacitor_SMD:C_0805_2012Metric" H 12238 5150 50  0001 C CNN
 F 3 "~" H 12200 5300 50  0001 C CNN
@@
 P 12200 5600
 F 0 "R6" H 12270 5646 50  0000 L CNN
-F 1 "R" H 12270 5555 50  0000 L CNN
+F 1 "5.1" H 12270 5555 50  0000 L CNN
 F 2 "Resistor_SMD:R_0805_2012Metric" V 12130 5600 50  0001 C CNN
 F 3 "~" H 12200 5600 50  0001 C CNN
@@
 P 8650 5400
 F 0 "C6" V 8398 5400 50  0000 C CNN
-F 1 "C" V 8489 5400 50  0000 C CNN
+F 1 ".22u" V 8489 5400 50  0000 C CNN
 F 2 "Capacitor_SMD:C_0805_2012Metric" H 8688 5250 50  0001 C CNN
 F 3 "~" H 8650 5400 50  0001 C CNN
@@
 P 11150 5400
 F 0 "C10" V 10898 5400 50  0000 C CNN
-F 1 "C" V 10989 5400 50  0000 C CNN
+F 1 ".22u" V 10989 5400 50  0000 C CNN
 F 2 "Capacitor_SMD:C_0805_2012Metric" H 11188 5250 50  0001 C CNN
 F 3 "~" H 11150 5400 50  0001 C CNN
@@
 P 6200 4650
 F 0 "R8" H 6270 4696 50  0000 L CNN
-F 1 "R" H 6270 4605 50  0000 L CNN
+F 1 "12" H 6270 4605 50  0000 L CNN
 F 2 "Resistor_SMD:R_0805_2012Metric" V 6130 4650 50  0001 C CNN
 F 3 "~" H 6200 4650 50  0001 C CNN
@@
 P 8950 4250
 F 0 "R11" H 9020 4296 50  0000 L CNN
-F 1 "R" H 9020 4205 50  0000 L CNN
+F 1 "12" H 9020 4205 50  0000 L CNN
 F 2 "Resistor_SMD:R_0805_2012Metric" V 8880 4250 50  0001 C CNN
 F 3 "~" H 8950 4250 50  0001 C CNN
@@
 P 6250 4850
 F 0 "R9" H 6320 4896 50  0000 L CNN
-F 1 "R" H 6320 4805 50  0000 L CNN
+F 1 "12" H 6320 4805 50  0000 L CNN
 F 2 "Resistor_SMD:R_0805_2012Metric" V 6180 4850 50  0001 C CNN
 F 3 "~" H 6250 4850 50  0001 C CNN
@@
 P 8950 5850
 F 0 "R12" H 9020 5896 50  0000 L CNN
-F 1 "R" H 9020 5805 50  0000 L CNN
+F 1 "12" H 9020 5805 50  0000 L CNN
 F 2 "Resistor_SMD:R_0805_2012Metric" V 8880 5850 50  0001 C CNN
 F 3 "~" H 8950 5850 50  0001 C CNN
@@
 P 11450 4250
 F 0 "R14" H 11520 4296 50  0000 L CNN
-F 1 "R" H 11520 4205 50  0000 L CNN
+F 1 "12" H 11520 4205 50  0000 L CNN
 F 2 "Resistor_SMD:R_0805_2012Metric" V 11380 4250 50  0001 C CNN
 F 3 "~" H 11450 4250 50  0001 C CNN
@@
 P 11450 5850
 F 0 "R15" H 11520 5896 50  0000 L CNN
-F 1 "R" H 11520 5805 50  0000 L CNN
+F 1 "12" H 11520 5805 50  0000 L CNN
 F 2 "Resistor_SMD:R_0805_2012Metric" V 11380 5850 50  0001 C CNN
 F 3 "~" H 11450 5850 50  0001 C CNN
@@
 P 5000 4150
 F 0 "R7" H 5070 4196 50  0000 L CNN
-F 1 "R" H 5070 4105 50  0000 L CNN
+F 1 "10" H 5070 4105 50  0000 L CNN
 F 2 "Resistor_SMD:R_0805_2012Metric" V 4930 4150 50  0001 C CNN
 F 3 "~" H 5000 4150 50  0001 C CNN
@@
 P 7700 5150
 F 0 "R10" H 7770 5196 50  0000 L CNN
-F 1 "R" H 7770 5105 50  0000 L CNN
+F 1 "10" H 7770 5105 50  0000 L CNN
 F 2 "Resistor_SMD:R_0805_2012Metric" V 7630 5150 50  0001 C CNN
 F 3 "~" H 7700 5150 50  0001 C CNN
@@
 P 10200 5150
 F 0 "R13" H 10270 5196 50  0000 L CNN
-F 1 "R" H 10270 5105 50  0000 L CNN
+F 1 "10" H 10270 5105 50  0000 L CNN
 F 2 "Resistor_SMD:R_0805_2012Metric" V 10130 5150 50  0001 C CNN
 F 3 "~" H 10200 5150 50  0001 C CNN
@@
 P 3950 5000
 F 0 "C14" H 3835 4954 50  0000 R CNN
-F 1 "C" H 3835 5045 50  0000 R CNN
+F 1 "100n" H 3835 5045 50  0000 R CNN
 F 2 "Capacitor_SMD:C_0805_2012Metric" H 3988 4850 50  0001 C CNN
 F 3 "~" H 3950 5000 50  0001 C CNN
@@
 P 3950 5550
 F 0 "C15" H 3835 5504 50  0000 R CNN
-F 1 "C" H 3835 5595 50  0000 R CNN
+F 1 "100n" H 3835 5595 50  0000 R CNN
 F 2 "Capacitor_SMD:C_0805_2012Metric" H 3988 5400 50  0001 C CNN
 F 3 "~" H 3950 5550 50  0001 C CNN
@@
 P 3950 6150
 F 0 "C16" H 3835 6104 50  0000 R CNN
-F 1 "C" H 3835 6195 50  0000 R CNN
+F 1 "100n" H 3835 6195 50  0000 R CNN
 F 2 "Capacitor_SMD:C_0805_2012Metric" H 3988 6000 50  0001 C CNN
 F 3 "~" H 3950 6150 50  0001 C CNN
