File: KiCAD_DRONE/Drone_rev0/ESC_rev1/ESC_rev1/ESC_rev1.kicad_pcb (KiCad board)
At the start: 2 copper layers, 34 parts, among them J1 Conn_01x02, J2 Conn_01x06, J3 Conn_01x05, Q1 IRF3205, Q2 IRF3205, Q3 IRF3205, Q4 IRF3205, Q5 IRF3205, Q6 IRF3205, U1 LM27222, U2 LM27222, U3 LM27222

Commit message: finished ESC rev1 layout!
Parts:
- added C14: C, Capacitor_SMD:C_0805_2012Metric, F.Cu at (99.6, 89.2)
- added C15: C, Capacitor_SMD:C_0805_2012Metric, F.Cu at (134.9, 88.9)
- added C16: C, Capacitor_SMD:C_0805_2012Metric, F.Cu at (165.7, 89.2)
- added J4: Conn_01x02, Connector_JST:JST_EH_B02B-EH-A_1x02_P2.50mm_Vertical, F.Cu at (100.8, 93.7)
- added J5: Conn_01x02, Connector_JST:JST_EH_B02B-EH-A_1x02_P2.50mm_Vertical, F.Cu at (136.1, 94.0)
- added J6: Conn_01x02, Connector_JST:JST_EH_B02B-EH-A_1x02_P2.50mm_Vertical, F.Cu at (167.1, 94.0)
- added R10: R, Resistor_SMD:R_0805_2012Metric, F.Cu at (134.6, 69.1)
- added R11: R, Resistor_SMD:R_0805_2012Metric, F.Cu at (147.7, 73.9)
- added R12: R, Resistor_SMD:R_0805_2012Metric, F.Cu at (147.5, 83.8)
- added R13: R, Resistor_SMD:R_0805_2012Metric, F.Cu at (164.3, 69.1)
- added R14: R, Resistor_SMD:R_0805_2012Metric, F.Cu at (174.4, 74.4)
- added R15: R, Resistor_SMD:R_0805_2012Metric, F.Cu at (175.3, 83.8)
- added R7: R, Resistor_SMD:R_0805_2012Metric, F.Cu at (98.7, 68.8)
- added R8: R, Resistor_SMD:R_0805_2012Metric, F.Cu at (115.9, 75.9)
- added R9: R, Resistor_SMD:R_0805_2012Metric, F.Cu at (116.0, 78.7)
- J3: value Conn_01x05 -> Conn_01x07; footprint Connector_PinHeader_2.54mm:PinHeader_1x05_P2.54mm_Vertical -> Connector_PinHeader_2.54mm:PinHeader_1x07_P2.54mm_Vertical
- moved J2 105.3 mm to (150.1, 55.4), turned to 270 degrees
- moved C1 73.0 mm to (142.7, 82.3), turned to 270 degrees
- moved C7 57.0 mm to (153.2, 68.1)
- moved J1 50.6 mm to (139.4, 83.6)
- moved C3 49.8 mm to (118.7, 67.6)
- moved J3 35.1 mm to (197.4, 75.2)
- moved C13 30.4 mm to (181.5, 68.3)
Connections:
- C1 pad 1: GND -> Vcc
- C1 pad 2: Vcc -> GND
- C5 pad 2: Net-(C5-Pad2) -> Net-(C2-Pad1)
- D1 pad 2: Vcc -> Net-(D1-Pad2)
- D2 pad 2: Vcc -> Net-(D2-Pad2)
- D3 pad 2: Vcc -> Net-(D3-Pad2)
- Q1 pad 3: Net-(C5-Pad2) -> Net-(C2-Pad1)
- Q2 pad 2: Net-(C5-Pad2) -> Net-(C2-Pad1)
- R1 pad 2: Net-(C5-Pad2) -> Net-(C2-Pad1)
- U1 pad 2: Net-(Q1-Pad1) -> Net-(R8-Pad2)
- U1 pad 6: Vcc -> Net-(D1-Pad2)
- U1 pad 7: Net-(Q2-Pad1) -> Net-(R9-Pad2)
- U1 pad 8: GND -> VSS1
- U2 pad 2: Net-(Q3-Pad1) -> Net-(R11-Pad2)
- U2 pad 6: Vcc -> Net-(D2-Pad2)
- U2 pad 7: Net-(Q4-Pad1) -> Net-(R12-Pad2)
- U2 pad 8: GND -> VSS2
- U3 pad 2: Net-(Q5-Pad1) -> Net-(R14-Pad2)
- U3 pad 6: Vcc -> Net-(D3-Pad2)
- U3 pad 7: Net-(Q6-Pad1) -> Net-(R15-Pad2)
- U3 pad 8: GND -> VSS3
Routing:
- net Net-(C2-Pad1): track 3.15 -> 107.0 mm, vias 0 -> 2
- net Net-(C6-Pad1): track 20.1 -> 71.5 mm, vias 0 -> 2
- net AH: track 0.00 -> 42.9 mm, vias 0 -> 1
- net AL: track 0.00 -> 41.3 mm, vias 0 -> 1
- net Net-(C10-Pad1): track 11.6 -> 44.9 mm, vias 0 -> 1
- net CL: track 0.00 -> 32.8 mm, vias 0 -> 1
- net CH: track 0.00 -> 32.0 mm
- net VDD3: track 0.00 -> 26.9 mm
- net VDD1: track 0.00 -> 25.4 mm
- net VDD2: track 0.00 -> 25.1 mm
- net VSS2: track 0.00 -> 23.9 mm
- net VSS1: track 0.00 -> 23.5 mm
- net VSS3: track 0.00 -> 23.1 mm
- net Net-(Q2-Pad1): track 23.0 -> 5.30 mm
- net Net-(R12-Pad2): track 0.00 -> 17.3 mm
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- added copper zone on F.Cu, net GND
- added copper zone on B.Cu, net Vcc
Other:
- board outline added: 106.7 x 45.7 mm

Commit message: added text and final layout changes. added m60 files.
Parts:
- J2: value Conn_01x06 -> Conn_01x07; footprint Connector_PinHeader_2.54mm:PinHeader_1x06_P2.54mm_Vertical -> Connector_JST:JST_EH_B07B-EH-A_1x07_P2.50mm_Vertical
- moved C1 21.9 mm to (131.5, 63.5)
- moved J1 21.9 mm to (128.2, 64.8)
- moved J2 2.30 mm to (152.4, 55.6), turned to 180 degrees
Connections:
- C15 pad 2: VSS2 -> VSS1
- C16 pad 2: VSS3 -> VSS1
- J2 pad 1: CH -> VSS1
- J2 pad 2: BH -> CH
- J2 pad 3: AH -> BH
- J2 pad 4: CL -> AH
- J2 pad 5: BL -> CL
- J2 pad 6: AL -> BL
- J5 pad 1: VSS2 -> VSS1
- J6 pad 1: VSS3 -> VSS1
- U2 pad 8: VSS2 -> VSS1
- U3 pad 8: VSS3 -> VSS1
Routing:
- net VSS1: track 23.5 -> 162.8 mm, vias 0 -> 4
- net VSS2: track 23.9 -> 0.00 mm
- net VSS3: track 23.1 -> 0.00 mm
- net GND: track 3.44 -> 0.00 mm
- net AH: track 42.9 -> 45.5 mm
- net CH: track 32.0 -> 30.9 mm
- net CL: track 32.8 -> 33.7 mm
- net Net-(D2-Pad2): track 9.47 -> 10.2 mm
- net Net-(R8-Pad2): track 13.6 -> 14.2 mm
Other:
- board size 106.7 x 45.7 mm -> 106.7 x 48.3 mm
- net class Default: clearance 0.2 -> 0.381; trace_width 0.25 -> 0.508
- net class everything added: clearance 0.381, trace_width 0.508, via_dia 0.8, via_drill 0.4
- rule trace_clearance: 0.2 -> 0.381
- rule trace_min: 0.2 -> 0.381
- board text added: "AVR ABC GND"
- board text added: "BLDC"
- board text added: "GD1"
- board text added: "GD2"
- board text added: "GD3"
- board text added: "GND"
- board text added: "PWR"
- board text added: "REV 0"
- board text added: "VCC"
