File: KiCAD_DRONE/Drone_rev0/ESC_rev0/ESC_rev0/ESC_rev0.sch (KiCad schematic (older format))
At the start: 49 parts, among them J1 Conn_01x02, J2 Conn_01x07, J3 Conn_01x07, J4 Conn_01x02, J5 Conn_01x02, J6 Conn_01x02, Q1 IRF3205, Q2 IRF3205, Q3 IRF3205, Q4 IRF3205, Q5 IRF3205, Q6 IRF3205, U1 LM27222, U2 LM27222, U3 LM27222

Commit message: renamed folders to appropriate revisions. created rev0.1 kicad project. this will contain common grounds bewteen gate driver and FETs.
Parts:
- C13: value 100u -> 100n
- U1, U2, U3: symbol My_Schematics:LM27222 -> ESC_rev1-rescue:LM27222-My_Schematics
Changed lines of the file:
@@
 $EndDescr
 $Comp
-L My_Schematics:LM27222 U1
+L ESC_rev1-rescue:LM27222-My_Schematics U1
 U 1 1 5CE9BBD8
 P 5250 4550
@@
 P 12250 3500
 F 0 "C13" H 12135 3454 50  0000 R CNN
-F 1 "100u" H 12135 3545 50  0000 R CNN
+F 1 "100n" H 12135 3545 50  0000 R CNN
 F 2 "Capacitor_SMD:C_0805_2012Metric" H 12288 3350 50  0001 C CNN
 F 3 "~" H 12250 3500 50  0001 C CNN
@@
 	3850 4050 4100 4050
 $Comp
-L My_Schematics:LM27222 U2
+L ESC_rev1-rescue:LM27222-My_Schematics U2
 U 1 1 5CEAE469
 P 7950 5550
@@
 	9100 5850 9100 5450
 $Comp
-L My_Schematics:LM27222 U3
+L ESC_rev1-rescue:LM27222-My_Schematics U3
 U 1 1 5CEBF7F5
 P 10450 5550
